Commit message: Renamed scout_mini.urdf.xacro to align with other files. Set wheel joint type to fixed.

File: scout_description/urdf/scout_wheel_type1.xacro (robot description, xacro)
@@ -49,5 +49,5 @@
             </collision>
         </link>
-        <joint name="${wheel_prefix}_wheel" type="continuous">
+        <joint name="${wheel_prefix}_wheel" type="fixed">
             <parent link="base_link"/>
             <child link="${wheel_prefix}_wheel_link"/>

File: scout_description/urdf/scout_wheel_type2.xacro (robot description, xacro)
@@ -49,5 +49,5 @@
             </collision>
         </link>
-        <joint name="${wheel_prefix}_wheel" type="continuous">
+        <joint name="${wheel_prefix}_wheel" type="fixed">
             <parent link="base_link"/>
             <child link="${wheel_prefix}_wheel_link"/>
